File: TC_SS.kicad_sch (KiCad schematic)
At the start: 35 parts, among them Q1 C2M0025120D, Q2 C2M0025120D, Q3 C2M0025120D, Q4 C2M0025120D, U1 IR2184, U2 IR2184, U3 SN74LVC1G14DBV, U4 SN74LVC1G14DBV, U5 NE555D

Commit message: Add some more values to components
Parts:
- C1, C2, C7: value C -> 100n
- C3, C5, C6: value C -> 330u
- C4: value C -> 330u'
- D1, D3: value D -> STTH2R06
- D4, D5, D6, D7: value D -> 1n4148
- R1, R2, R3, R4: value R -> 22
Other:
- moved on the sheet: C9
