File: TC_SS.kicad_sch (KiCad schematic)
At the start: 58 parts, among them IC1 ADUM4221-1ARIZ, IC2 ADUM4221-1ARIZ, J1 15V_In, Q1 IPW60R099P6XKSA1, Q2 IPW60R099P6XKSA1, Q3 IPW60R099P6XKSA1, Q4 IPW60R099P6XKSA1, U1 LM7805_TO220, U2 74HC14, U3 LM7812_TO220

Commit message: Almost ready to produce
Parts:
- added C20, C21, C22, C23, C28, C29, C30, C31, C32, C33, C36, C37, C38, C39: 1u, Capacitor_SMD:C_0805_2012Metric, symbol Device:C_Small
- added C24, C25, C26, C27, C34, C35: 100n, Capacitor_SMD:C_0805_2012Metric, symbol Device:C_Small
- added H1, H2, H3, H4: MountingHole_Pad, MountingHole:MountingHole_3.2mm_M3_Pad_Via, symbol Mechanical:MountingHole_Pad
- added J2, J3, J4, J5, J6: Conn_Coaxial, Connector_Coaxial:SMA_Samtec_SMA-J-P-X-ST-EM1_EdgeMount, symbol Connector:Conn_Coaxial
- added TP1, TP2: TestPoint, TestPoint:TestPoint_Loop_D3.50mm_Drill1.4mm_Beaded, symbol Connector:TestPoint
- C10, C4: value 1u -> 10u
- D1, D4, D5, D6: value D -> DFLS120L-7
- R5, R6: value 10k -> 22
- U2: footprint (none) -> SamacSys_Parts:SOIC127P600X175-14N
Connections:
- net +12V: now also PS3.1 (+VIN), C36.2, C37.1, C38.1, C39.2
- net GND: now also #T1.3 (SA), D3.2 (A), PS3.2 (-VIN), C20.2, C21.1, C24.2, C25.1, C32.2, C33.1, C34.2, C35.1, C36.1, C37.2, C38.2, C39.1, H1.1, H2.1, H3.1, H4.1, J2.2 (Ext), J3.2 (Ext), J4.2 (Ext), J5.2 (Ext), J6.2 (Ext), TP1.1
- net HB1: now also C22.2, C23.1, C26.1, C27.2
- net HB2: now also PS3.6 (NO_PIN), C28.2, C29.1, C30.2, C31.1
- net HS1_G: now also D6.2 (A); no longer D6.1 (K)
- net LS1_G: now also D5.2 (A); no longer D5.1 (K)
- net PWM: now also J2.1 (In); no longer IC1.1 (PWM), IC2.1 (PWM)
- net Vg_neg_HS1: now also C23.2, C26.2
- net Vg_neg_HS2: now also PS3.5 (-VOUT), C29.2, C31.2
- net Vg_neg_LS1: now also C21.2, C25.2
- net Vg_neg_LS2: now also C33.2, C35.2
- net Vg_pos_HS1: now also C22.1, C27.1
- net Vg_pos_HS2: now also PS3.7 (+VOUT), C28.1, C30.1
- net Vg_pos_LS1: now also C20.1, C24.1
- net Vg_pos_LS2: now also C32.1, C34.1
- net at #T1.4 (SB), R10.1: now also TP2.1
- net at IC1.10 (VOB), R6.1: now also D5.1 (K); no longer D5.2 (A)
- net at IC1.15 (VOA), R5.1: now also D6.1 (K); no longer D6.2 (A)
- net at IC1.5 (DISABLE): now also J4.1 (In)
- net at IC2.5 (DISABLE): now also J6.1 (In)
- new net: IC1.1 (PWM), J3.1 (In)
- new net: IC2.1 (PWM), J5.1 (In)
Other:
- moved on the sheet: D5, D6, PS1, PS2, PS3

Commit message: Done now (probably)
Parts:
- C30, C31: value 1u -> 100n
Changed lines of the file:
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@@
       (effects (font (size 1.27 1.27)) (justify left))
     )
-    (property "Value" "1u" (at 220.98 71.1263 0)
+    (property "Value" "100n" (at 220.98 71.1263 0)
       (effects (font (size 1.27 1.27)) (justify left))
     )
@@
       (effects (font (size 1.27 1.27)) (justify left))
     )
-    (property "Value" "1u" (at 220.98 76.2063 0)
-      (effects (font (size 1.27 1.27)) (justify left))
-    )
+    (property "Value" "100n" (at 220.98 76.2063 0)
+      (effects (font (size 1.27 1.27)) (justify left))
+    )
