File: powersupply.kicad_sch (KiCad schematic)
At the start: 7 parts

Commit message: Update Power PCB
Parts:
- C3, C4, C5, C6: footprint Capacitor_THT:C_Radial_D8.0mm_H11.5mm_P3.50mm -> Capacitor_THT:CP_Radial_D35.0mm_P10.00mm_SnapIn
Changed lines of the file:
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@@
       (effects (font (size 1.27 1.27)) (justify left))
     )
-    (property "Footprint" "Capacitor_THT:C_Radial_D8.0mm_H11.5mm_P3.50mm" (at 148.2852 100.33 0)
+    (property "Footprint" "Capacitor_THT:CP_Radial_D35.0mm_P10.00mm_SnapIn" (at 148.2852 100.33 0)
       (effects (font (size 1.27 1.27)) hide)
     )
@@
       (effects (font (size 1.27 1.27)) (justify left))
     )
-    (property "Footprint" "Capacitor_THT:C_Radial_D8.0mm_H11.5mm_P3.50mm" (at 166.0652 100.33 0)
+    (property "Footprint" "Capacitor_THT:CP_Radial_D35.0mm_P10.00mm_SnapIn" (at 166.0652 100.33 0)
       (effects (font (size 1.27 1.27)) hide)
     )
@@
       (effects (font (size 1.27 1.27)) (justify left))
     )
-    (property "Footprint" "Capacitor_THT:C_Radial_D8.0mm_H11.5mm_P3.50mm" (at 157.1752 100.33 0)
+    (property "Footprint" "Capacitor_THT:CP_Radial_D35.0mm_P10.00mm_SnapIn" (at 157.1752 100.33 0)
       (effects (font (size 1.27 1.27)) hide)
     )
@@
       (effects (font (size 1.27 1.27)) (justify left))
     )
-    (property "Footprint" "Capacitor_THT:C_Radial_D8.0mm_H11.5mm_P3.50mm" (at 174.9552 100.33 0)
+    (property "Footprint" "Capacitor_THT:CP_Radial_D35.0mm_P10.00mm_SnapIn" (at 174.9552 100.33 0)
       (effects (font (size 1.27 1.27)) hide)
     )
